File: pcb/driver_board/driver_board.kicad_sch (KiCad schematic)
At the start: 23 parts, among them J1 Conn_ARM_JTAG_SWD_20, J2 Barrel_Jack, J3 USB_C_Receptacle_PowerOnly_6P, SW1 SW_SPDT, U2 STM32H755ZITx

Commit message: start adding wifi connectivity
Parts:
- removed SW1: SW_SPDT, symbol Switch:SW_SPDT
- added D5: PRTR5V0U4D,125, SOT95P275X110-6N, symbol PRTR5V0U4D_125:PRTR5V0U4D,125
- added R5, R6: R_US, symbol Device:R_US
- added R7, R8: 0R, symbol Device:R_US
- added SW2: SW_MEC_5G, symbol Switch:SW_MEC_5G
- added U1: NCV1117ST33T3G, SOT223-3_ONS, symbol 2025-08-29_01-45-15:NCV1117ST33T3G
- added Y1, Y2: Crystal, symbol Device:Crystal
Connections:
- net VDD_MCU is gone; now on net VDDA: C1.1, C10.1, C11.1, C2.1, C3.1, C4.1, C5.1, C6.1, C7.1, C8.1, C9.1, U2.106 (VDD), U2.119 (VDD), U2.129 (VDD), U2.13 (VDD), U2.144 (VDD), U2.19 (VDD), U2.32 (VDD), U2.42 (VDD), U2.56 (VDD), U2.7 (VDD), U2.71 (VDD), U2.79 (VDD), U2.8 (VBAT), U2.92 (VDD)
- net +3V3: now also SW2.1 (A), SW2.2 (A)
- net GND: now also J1.1 (VTREF), U2.104 (VSS), U2.118 (VSS), U2.12 (VSS), U2.128 (VSS), U2.141 (VSS), U2.18 (VSS), U2.33 (VSS), U2.41 (VSS), U2.55 (VSS), U2.6 (VSS), U2.69 (VSS), U2.80 (VSS), U2.89 (VSS), R5.2
- net OSC_32_IN: now reaches U2.10 (PC14)
- net at U2.102 (PA13): no longer J1.7 (TMS/SWDIO)
- net at U2.107 (PA14): no longer J1.9 (TCK/SWCLK)
- net at U2.108 (PA15): no longer J1.5 (TDI)
- net OSC_32_OUT: now reaches U2.11 (PC15)
- net at U2.130 (PB3): no longer J1.13 (TDO/SWO)
- net at U2.131 (PB4): no longer J1.3 (~{TRST})
- net VDDA: now reaches U2.35 (VREF+)
- net VDDA: now also U2.36 (VDDA)
- new net: R8.2, Y2.2
- new net: D5.1 (I/O1), J1.5 (TDI)
- new net: SW2.3 (B), SW2.4 (B)
- new net: R7.2, Y2.1
- new net: D5.2 (GND), R5.1
- new net VDD: R6.2
Other:
- added sheet PoE (PoE.kicad_sch)
- added sheet WiFi Connectivity (wifi.kicad_sch)
- note added: "External HSE Source(Optional)"
- note added: "External LSE source"
- note added: "PDN decoupling"
- moved on the sheet: C1, C10, C11, C2, C3, C4, C5, C6, C7, C8, C9, J1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
